File: kastenwagen-1840-chunky/kastenwagen-1840-chunky.kicad_pcb (KiCad board)
At the start: 2 copper layers, 350.5 x 83.5 mm, 109 parts, among them U2 Helios

Commit message: Silkscreen update
Other:
- board text added: "Kastenwagen PCB Chunky NoPunIn10Did Port by exen904 RP2040 Prototype 2024-12"
- board text removed: "Kastenwagen PCB Chunky NoPunIn10Did Prototype 2023-04"
Changed lines of the file:
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@@
 		)
 	)
-	(gr_text "Kastenwagen PCB Chunky\nNoPunIn10Did\nPrototype 2023-04"
+	(gr_text "Kastenwagen PCB Chunky\nNoPunIn10Did Port by exen904\nRP2040 Prototype 2024-12"
 		(at 229.39375 89.69375 0)
 		(layer "F.SilkS")
